Commit message: working now on urdf safe

File: rl_deploy/spot_with_arm.urdf (robot description, URDF)
Before this commit: robot spot_with_arm, 9 links, 8 joints
Links:
- added link fl_foot; collision sphere radius=0.036
- added link fl_hip, mass 1.13688339; visual mesh filename=meshes/base/visual/front_left_hip.obj
- added link fl_lleg, mass 0.330; collision mesh filename=meshes/base/collision/lower_leg_collision.obj; visual mesh filename=meshes/base/visual/front_left_lower_leg.obj
- added link fl_uleg, mass 2.25620359; collision mesh filename=meshes/base/collision/upper_leg_collision.obj; visual mesh filename=meshes/base/visual/front_left_upper_leg.obj
- added link fr_foot; collision sphere radius=0.036
- added link fr_hip, mass 1.13688339; visual mesh filename=meshes/base/visual/front_right_hip.obj
- added link fr_lleg, mass 0.330; collision mesh filename=meshes/base/collision/lower_leg_collision.obj; visual mesh filename=meshes/base/visual/front_right_lower_leg.obj
- added link fr_uleg, mass 2.25620359; collision mesh filename=meshes/base/collision/upper_leg_collision.obj; visual mesh filename=meshes/base/visual/front_right_upper_leg.obj
- added link hl_foot; collision sphere radius=0.036
- added link hl_hip, mass 1.13688339; visual mesh filename=meshes/base/visual/rear_left_hip.obj
- added link hl_lleg, mass 0.330; collision mesh filename=meshes/base/collision/lower_leg_collision.obj; visual mesh filename=meshes/base/visual/rear_left_lower_leg.obj
- added link hl_uleg, mass 2.25620359; collision mesh filename=meshes/base/collision/upper_leg_collision.obj; visual mesh filename=meshes/base/visual/rear_left_upper_leg.obj
- added link hr_foot; collision sphere radius=0.036
- added link hr_hip, mass 1.13688339; visual mesh filename=meshes/base/visual/rear_right_hip.obj
- added link hr_lleg, mass 0.330; collision mesh filename=meshes/base/collision/lower_leg_collision.obj; visual mesh filename=meshes/base/visual/rear_right_lower_leg.obj
- added link hr_uleg, mass 2.25620359; collision mesh filename=meshes/base/collision/upper_leg_collision.obj; visual mesh filename=meshes/base/visual/rear_right_upper_leg.obj
- link arm_link_el0: geometry visual mesh filename=meshes/arm/visual/arm_link_el0.obj
- link arm_link_sh0: geometry visual mesh filename=meshes/arm/visual/arm_link_sh0.obj
- link arm_link_wr0: geometry visual mesh filename=meshes/arm/visual/arm_link_wr0.obj
Joints:
- added joint fl_ank: type fixed, parent fl_lleg, child fl_foot, origin xyz=0.0 0.0 -0.3365
- added joint fl_hx: type revolute, parent body, child fl_hip, origin xyz=0.29785 0.05500 0.00000 rpy=0 0 0, axis 1 0 0, limit lower=-0.785398 upper=0.785398 effort=45 velocity=100
- added joint fl_hy: type revolute, parent fl_hip, child fl_uleg, origin xyz=0.0 0.110945 0.0 rpy=0 0 0, axis 0 1 0, limit lower=-0.898845 upper=2.295108 effort=45 velocity=100
- added joint fl_kn: type revolute, parent fl_uleg, child fl_lleg, origin xyz=0.025 0.000 -0.3205 rpy=0 0 0, axis 0 1 0, limit lower=-2.7929 upper=-0.2471 effort=115 velocity=100
- added joint fr_ank: type fixed, parent fr_lleg, child fr_foot, origin xyz=0.0 0.0 -0.3365
- added joint fr_hx: type revolute, parent body, child fr_hip, origin xyz=0.29785 -0.05500 0.00000 rpy=0 0 0, axis 1 0 0, limit lower=-0.785398 upper=0.785398 effort=45 velocity=100
- added joint fr_hy: type revolute, parent fr_hip, child fr_uleg, origin xyz=0.0 -0.110945 0.0 rpy=0 0 0, axis 0 1 0, limit lower=-0.898845 upper=2.295108 effort=45 velocity=100
- added joint fr_kn: type revolute, parent fr_uleg, child fr_lleg, origin xyz=0.025 0.000 -0.3205 rpy=0 0 0, axis 0 1 0, limit lower=-2.7929 upper=-0.2471 effort=115 velocity=100
- added joint hl_ank: type fixed, parent hl_lleg, child hl_foot, origin xyz=0.0 0.0 -0.3365
- added joint hl_hx: type revolute, parent body, child hl_hip, origin xyz=-0.29785 0.05500 0.00000 rpy=0 0 0, axis 1 0 0, limit lower=-0.785398 upper=0.785398 effort=45 velocity=100
- added joint hl_hy: type revolute, parent hl_hip, child hl_uleg, origin xyz=0.0 0.110945 0.0 rpy=0 0 0, axis 0 1 0, limit lower=-0.898845 upper=2.295108 effort=45 velocity=100
- added joint hl_kn: type revolute, parent hl_uleg, child hl_lleg, origin xyz=0.025 0.000 -0.3205 rpy=0 0 0, axis 0 1 0, limit lower=-2.7929 upper=-0.2471 effort=115 velocity=100
- added joint hr_ank: type fixed, parent hr_lleg, child hr_foot, origin xyz=0.0 0.0 -0.3365
- added joint hr_hx: type revolute, parent body, child hr_hip, origin xyz=-0.29785 -0.05500 0.00000 rpy=0 0 0, axis 1 0 0, limit lower=-0.785398 upper=0.785398 effort=45 velocity=100
- added joint hr_hy: type revolute, parent hr_hip, child hr_uleg, origin xyz=0.0 -0.110945 0.0 rpy=0 0 0, axis 0 1 0, limit lower=-0.898845 upper=2.295108 effort=45 velocity=100
- added joint hr_kn: type revolute, parent hr_uleg, child hr_lleg, origin xyz=0.025 0.000 -0.3205 rpy=0 0 0, axis 0 1 0, limit lower=-2.7929 upper=-0.2471 effort=115 velocity=100
- joint arm_el0: limit lower=0 upper=3.14159 effort=90.9 velocity=100 -> lower=0 upper=3.14159 effort=204.5 velocity=100
- joint arm_el1: limit lower=-2.792530 upper=2.792530 effort=30.3 velocity=100 -> lower=-2.792530 upper=2.792530 effort=102 velocity=100
- joint arm_jaw: limit (none) -> lower=-1.5708 upper=0.0 effort=15.32 velocity=100
- joint arm_sh0: limit lower=-2.61799 upper=3.14159 effort=90.9 velocity=100 -> lower=-2.61799 upper=3.14159 effort=1020 velocity=100
- joint arm_sh1: limit lower=-3.14159 upper=0.523599 effort=181.8 velocity=100 -> lower=-3.14159 upper=0.523599 effort=255 velocity=100
- joint arm_wr0: limit lower=-1.8326 upper=1.8326 effort=30.3 velocity=100 -> lower=-1.8326 upper=1.8326 effort=102 velocity=100
- joint arm_wr1: limit lower=-2.87989 upper=2.87979 effort=30.3 velocity=100 -> lower=-2.87989 upper=2.87979 effort=102 velocity=100
